Commit message: New configuration for the joint calibration of the PR2

File: tams_pr2_atom_calibration/urdf/optimized.urdf.xacro (robot description, xacro)
@@ -1535,16 +1535,22 @@
   </link>
   <joint name="azure_kinect_camera_base_to_rgb_sensor_joint" type="fixed">
-    <origin xyz="-0.01792 -0.032 0.0" rpy="0.0 0.0 0.0"/>
+    <origin xyz="-0.006087549382002858 -0.029180110849404146 0.002963802698343846" rpy="-0.011639277151118984 -0.023149641698049925 -0.003980766965896363"/>
     <parent link="azure_kinect_camera_base"/>
     <child link="azure_kinect_rgb_sensor"/>
   </joint>
-  <link name="azure_kinect_rgb_camera_link_urdf"/>
+  <link name="azure_kinect_rgb_camera_link"/>
   <joint name="azure_kinect_rgb_sensor_to_rgb_camera_joint" type="fixed">
     <origin xyz="0.01411221072129154 -5.274945064383946e-05 -0.00025686822127624076" rpy="-1.576436 0.0016804 -1.5680018"/>
     <parent link="azure_kinect_rgb_sensor"/>
-    <child link="azure_kinect_rgb_camera_link_urdf"/>
+    <child link="azure_kinect_rgb_camera_link"/>
+  </joint>
+  <link name="azure_kinect_depth_camera_link"/>
+  <joint name="azure_kinect_depth_sensor_to_depth_camera_joint" type="fixed">
+    <origin xyz="0.01411221072129154 -5.274945064383946e-05 -0.00025686822127624076" rpy="-1.576436 0.0016804 -1.5680018"/>
+    <parent link="azure_kinect_depth_sensor"/>
+    <child link="azure_kinect_depth_camera_link"/>
   </joint>
   <joint name="azure_kinect_camera_base_joint" type="fixed">
-    <origin xyz="0.05326841953691841 0.006597606436255618 0.17424594407306315" rpy="0.007285055140918984 0.08145909946609553 0.02776856447767072"/>
+    <origin xyz="0.048 0.0 0.171" rpy="0.0 0.0 0.0"/>
     <parent link="head_plate_frame"/>
     <child link="azure_kinect_camera_base"/>

File: tams_pr2_description/urdf/tams_azure_kinect.urdf.xacro (robot description, xacro)
@@ -146,9 +146,16 @@
   The real ${name}_rgb_camera_link is published by the azure from its internal calibration.
   The link here should use the same calibration (extracted via TF) and is required for robot_calibration
+  This is the same for ATOM calibration
   -->
-  <link name="${name}_rgb_camera_link_urdf" />
+  <link name="${name}_rgb_camera_link" />
   <joint name="${name}_rgb_sensor_to_rgb_camera_joint" type="fixed">
     <parent link="${name}_rgb_sensor" />
-    <child link="${name}_rgb_camera_link_urdf" />
+    <child link="${name}_rgb_camera_link" />
+    <origin xyz="0.01411221072129154 -5.274945064383946e-05 -0.00025686822127624076" rpy="-1.576436 0.0016804 -1.5680018" />
+  </joint>
+  <link name="${name}_depth_camera_link" />
+  <joint name="${name}_depth_sensor_to_depth_camera_joint" type="fixed">
+    <parent link="${name}_depth_sensor" />
+    <child link="${name}_depth_camera_link" />
     <origin xyz="0.01411221072129154 -5.274945064383946e-05 -0.00025686822127624076" rpy="-1.576436 0.0016804 -1.5680018" />
   </joint>

Commit message: New optimized urdf with big dataset and upload pr2 updated

File: tams_pr2_atom_calibration/urdf/optimized.urdf.xacro (robot description, xacro)
@@ -918,5 +918,5 @@
     <dynamics damping="0.5"/>
     <safety_controller k_velocity="1.5" k_position="100.0" soft_lower_limit="-2.857" soft_upper_limit="2.857"/>
-    <calibration rising="0.0303234" falling="0"/>
+    <calibration rising="0.01531154062790617" falling="0"/>
   </joint>
   <link name="head_pan_link">
@@ -956,5 +956,5 @@
     <dynamics damping="10.0"/>
     <safety_controller k_velocity="3.0" k_position="100.0" soft_lower_limit="-0.3712" soft_upper_limit="1.29626"/>
-    <calibration rising="0" falling="0.0110223"/>
+    <calibration rising="0" falling="-8.577235131254635e-05"/>
   </joint>
   <link name="head_tilt_link">
@@ -1535,5 +1535,5 @@
   </link>
   <joint name="azure_kinect_camera_base_to_rgb_sensor_joint" type="fixed">
-    <origin xyz="-0.006087549382002858 -0.029180110849404146 0.002963802698343846" rpy="-0.011639277151118984 -0.023149641698049925 -0.003980766965896363"/>
+    <origin xyz="-0.01792 -0.032 0.0" rpy="0.0 0.0 0.0"/>
     <parent link="azure_kinect_camera_base"/>
     <child link="azure_kinect_rgb_sensor"/>
@@ -1552,5 +1552,5 @@
   </joint>
   <joint name="azure_kinect_camera_base_joint" type="fixed">
-    <origin xyz="0.048 0.0 0.171" rpy="0.0 0.0 0.0"/>
+    <origin xyz="0.05156534529647598 0.002670728318304638 0.1777151884004853" rpy="-0.00808453173647982 -0.014528287360892594 -0.0014224511549819012"/>
     <parent link="head_plate_frame"/>
     <child link="azure_kinect_camera_base"/>
@@ -3584,5 +3584,5 @@
     <dynamics damping="10.0"/>
     <safety_controller k_velocity="10.0" k_position="100.0" soft_lower_limit="-0.5646018366025517" soft_upper_limit="2.1353981633974484"/>
-    <calibration rising="0.82713499" falling="0"/>
+    <calibration rising="0.8134834214597091" falling="0"/>
   </joint>
   <link name="l_shoulder_pan_link">
@@ -3614,5 +3614,5 @@
     <dynamics damping="10.0"/>
     <safety_controller k_velocity="10.0" k_position="100.0" soft_lower_limit="-0.3535999999999999" soft_upper_limit="1.2963"/>
-    <calibration rising="0" falling="0.029331549999999998"/>
+    <calibration rising="0" falling="-0.003869385516868981"/>
   </joint>
   <link name="l_shoulder_lift_link">
@@ -3644,5 +3644,5 @@
     <dynamics damping="0.1"/>
     <safety_controller k_velocity="2.0" k_position="100.0" soft_lower_limit="-0.65" soft_upper_limit="3.7500000000000004"/>
-    <calibration rising="1.6001292999999999" falling="0"/>
+    <calibration rising="1.593225178979538" falling="0"/>
   </joint>
   <link name="l_upper_arm_roll_link">
@@ -3752,5 +3752,5 @@
     <dynamics damping="0.1"/>
     <safety_controller k_velocity="1.0" k_position="0" soft_lower_limit="0" soft_upper_limit="0"/>
-    <calibration rising="0.063877" falling="0"/>
+    <calibration rising="0.014317360556922419" falling="0"/>
   </joint>
   <link name="l_forearm_roll_link">
@@ -3798,5 +3798,5 @@
     <dynamics damping="1.0"/>
     <safety_controller k_velocity="3.0" k_position="100.0" soft_lower_limit="-2.1212999999999997" soft_upper_limit="-0.15"/>
-    <calibration rising="0" falling="-1.3127588"/>
+    <calibration rising="0" falling="-1.3069393634533952"/>
   </joint>
   <link name="l_elbow_flex_link">
@@ -3869,5 +3869,5 @@
     <dynamics damping="0.1"/>
     <safety_controller k_velocity="4.0" k_position="20.0" soft_lower_limit="-2.0" soft_upper_limit="-0.1"/>
-    <calibration rising="0" falling="-0.5442714999999999"/>
+    <calibration rising="0" falling="-0.5284454525275436"/>
   </joint>
   <link name="l_wrist_flex_link">
@@ -3899,5 +3899,5 @@
     <dynamics damping="0.1"/>
     <safety_controller k_velocity="2.0" k_position="0" soft_lower_limit="0" soft_upper_limit="0"/>
-    <calibration rising="-1.49252392" falling="0"/>
+    <calibration rising="-1.4549082745368125" falling="0"/>
   </joint>
   <link name="l_wrist_roll_link">

Commit message: Optimized URDF for robot deployment

File: tams_pr2_atom_calibration/urdf/optimized.urdf.xacro (robot description, xacro)
@@ -918,5 +918,5 @@
     <dynamics damping="0.5"/>
     <safety_controller k_velocity="1.5" k_position="100.0" soft_lower_limit="-2.857" soft_upper_limit="2.857"/>
-    <calibration rising="0.01531154062790617" falling="0"/>
+    <calibration rising="0.0303234" falling="0"/>
   </joint>
   <link name="head_pan_link">
@@ -956,5 +956,5 @@
     <dynamics damping="10.0"/>
     <safety_controller k_velocity="3.0" k_position="100.0" soft_lower_limit="-0.3712" soft_upper_limit="1.29626"/>
-    <calibration rising="0" falling="-8.577235131254635e-05"/>
+    <calibration rising="0" falling="0.0110223"/>
   </joint>
   <link name="head_tilt_link">
@@ -1535,5 +1535,5 @@
   </link>
   <joint name="azure_kinect_camera_base_to_rgb_sensor_joint" type="fixed">
-    <origin xyz="-0.01792 -0.032 0.0" rpy="0.0 0.0 0.0"/>
+    <origin xyz="-0.014227721190625557 -0.03557117609122215 0.0062478521987937435" rpy="0.0037205293142486195 -0.025777618872663086 -0.001500255392035359"/>
     <parent link="azure_kinect_camera_base"/>
     <child link="azure_kinect_rgb_sensor"/>
@@ -1552,5 +1552,5 @@
   </joint>
   <joint name="azure_kinect_camera_base_joint" type="fixed">
-    <origin xyz="0.05156534529647598 0.002670728318304638 0.1777151884004853" rpy="-0.00808453173647982 -0.014528287360892594 -0.0014224511549819012"/>
+    <origin xyz="0.048 0.0 0.171" rpy="0.0 0.0 0.0"/>
     <parent link="head_plate_frame"/>
     <child link="azure_kinect_camera_base"/>
@@ -3584,5 +3584,5 @@
     <dynamics damping="10.0"/>
     <safety_controller k_velocity="10.0" k_position="100.0" soft_lower_limit="-0.5646018366025517" soft_upper_limit="2.1353981633974484"/>
-    <calibration rising="0.8134834214597091" falling="0"/>
+    <calibration rising="0.8292206191927028" falling="0"/>
   </joint>
   <link name="l_shoulder_pan_link">
@@ -3614,5 +3614,5 @@
     <dynamics damping="10.0"/>
     <safety_controller k_velocity="10.0" k_position="100.0" soft_lower_limit="-0.3535999999999999" soft_upper_limit="1.2963"/>
-    <calibration rising="0" falling="-0.003869385516868981"/>
+    <calibration rising="0" falling="0.007359737698904842"/>
   </joint>
   <link name="l_shoulder_lift_link">
@@ -3644,5 +3644,5 @@
     <dynamics damping="0.1"/>
     <safety_controller k_velocity="2.0" k_position="100.0" soft_lower_limit="-0.65" soft_upper_limit="3.7500000000000004"/>
-    <calibration rising="1.593225178979538" falling="0"/>
+    <calibration rising="1.6052983922691766" falling="0"/>
   </joint>
   <link name="l_upper_arm_roll_link">
@@ -3752,5 +3752,5 @@
     <dynamics damping="0.1"/>
     <safety_controller k_velocity="1.0" k_position="0" soft_lower_limit="0" soft_upper_limit="0"/>
-    <calibration rising="0.014317360556922419" falling="0"/>
+    <calibration rising="0.009442019548690957" falling="0"/>
   </joint>
   <link name="l_forearm_roll_link">
@@ -3798,5 +3798,5 @@
     <dynamics damping="1.0"/>
     <safety_controller k_velocity="3.0" k_position="100.0" soft_lower_limit="-2.1212999999999997" soft_upper_limit="-0.15"/>
-    <calibration rising="0" falling="-1.3069393634533952"/>
+    <calibration rising="0" falling="-1.3054432621075143"/>
   </joint>
   <link name="l_elbow_flex_link">
@@ -3869,5 +3869,5 @@
     <dynamics damping="0.1"/>
     <safety_controller k_velocity="4.0" k_position="20.0" soft_lower_limit="-2.0" soft_upper_limit="-0.1"/>
-    <calibration rising="0" falling="-0.5284454525275436"/>
+    <calibration rising="0" falling="-0.5260047455156464"/>
   </joint>
   <link name="l_wrist_flex_link">
@@ -3899,5 +3899,5 @@
     <dynamics damping="0.1"/>
     <safety_controller k_velocity="2.0" k_position="0" soft_lower_limit="0" soft_upper_limit="0"/>
-    <calibration rising="-1.4549082745368125" falling="0"/>
+    <calibration rising="-1.5351463737705227" falling="0"/>
   </joint>
   <link name="l_wrist_roll_link">
