Commit message: Updating TAMS PR2 atom calibration
Adding a README.md and last updates to the atom calibration package

File: tams_pr2_atom_calibration/urdf/initial_estimate.urdf.xacro (robot description, xacro)
@@ -120,4 +120,35 @@
     <origin xyz="0 0 0" rpy="0 1.5707963267948966 -1.2217304763960306" />
   </xacro:pr2_gripper_v0>
+  <!-- Add cyllinder for touch experiment -->
+  <xacro:property name="cylinder_radius" value="0.002" />
+  <xacro:property name="cylinder_length" value="0.02099" />
+  <joint name="touch_probe_cylinder_base_joint" type="fixed">
+    <origin xyz="0.019 0 0" rpy="0 0 0" />
+    <parent link="l_gripper_tool_frame"/>
+    <child link="touch_probe_cylinder_base_frame"/>
+  </joint>
+  <link name="touch_probe_cylinder_base_frame"/>
+  <joint name="touch_probe_cylinder_top_joint" type="fixed">
+    <origin xyz="${cylinder_length} 0 0" rpy="0 0 0" />
+    <parent link="touch_probe_cylinder_base_frame"/>
+    <child link="touch_probe_cylinder_top_frame"/>
+  </joint>
+  <link name="touch_probe_cylinder_top_frame">
+   <visual>
+     <origin xyz="${-cylinder_length/2} 0 0" rpy="0 ${-M_PI/2} 0" />
+     <geometry>
+       <cylinder radius="${cylinder_radius}" length="${cylinder_length}"/>
+     </geometry>
+     <material name="Grey">
+       <color rgba="0.5 0.5 0.5 1.0"/>
+     </material>
+   </visual>
+   <collision>
+     <origin xyz="${-cylinder_length/2} 0 0" rpy="0 ${-M_PI/2} 0" />
+     <geometry>
+       <cylinder radius="${cylinder_radius}" length="${cylinder_length}"/>
+     </geometry>
+   </collision>
+  </link>
   <!-- Forearm cam Position is a guess, based on full robot calibration -->
   <!-- Forearm cam Orientation is from Function -->

File: tams_pr2_atom_calibration/urdf/optimized_manual_adjust.urdf.xacro (robot description, xacro)
@@ -911,5 +911,5 @@
   </gazebo>
   <joint name="head_pan_joint" type="revolute">
-    <origin xyz="-0.01707 0.0 0.38145" rpy="0.0 0.0 -0.03897654545492374"/>
+    <origin xyz="-0.01707 0.0 0.38145" rpy="0.0 0.0 0.0"/>
     <axis xyz="0.0 0.0 1.0"/>
     <parent link="torso_lift_link"/>
@@ -918,5 +918,5 @@
     <dynamics damping="0.5"/>
     <safety_controller k_velocity="1.5" k_position="100.0" soft_lower_limit="-2.857" soft_upper_limit="2.857"/>
-    <calibration rising="0.0521899521255305" falling="0"/>
+    <calibration rising="0.0303234" falling="0"/>
   </joint>
   <link name="head_pan_link">
@@ -949,5 +949,5 @@
   </transmission>
   <joint name="head_tilt_joint" type="revolute">
-    <origin xyz="0.068 0.0 0.0" rpy="0.0 -0.025225546349730715 0.0"/>
+    <origin xyz="0.068 0.0 0.0" rpy="0.0 0.0 0.0"/>
     <axis xyz="0.0 1.0 0.0"/>
     <parent link="head_pan_link"/>
@@ -956,5 +956,5 @@
     <dynamics damping="10.0"/>
     <safety_controller k_velocity="3.0" k_position="100.0" soft_lower_limit="-0.3712" soft_upper_limit="1.29626"/>
-    <calibration rising="0" falling="0.05047299239962615"/>
+    <calibration rising="0" falling="0.0110223"/>
   </joint>
   <link name="head_tilt_link">
@@ -1535,5 +1535,5 @@
   </link>
   <joint name="azure_kinect_camera_base_to_rgb_sensor_joint" type="fixed">
-    <origin xyz="-0.07466568353559286 -0.03210135506543399 -0.012904341249372842" rpy="-0.0056235786454332665 0.005404129792773083 0.008111063480687923"/>
+    <origin xyz="-0.01721323301495916 -0.02901985231172751 0.009946408323916658" rpy="-0.007722464822759145 -0.025976485755276633 -0.0070823237921861645"/>
     <parent link="azure_kinect_camera_base"/>
     <child link="azure_kinect_rgb_sensor"/>
@@ -1552,5 +1552,5 @@
   </joint>
   <joint name="azure_kinect_camera_base_joint" type="fixed">
-    <origin xyz="0.04797663865993433 -0.008366640694689446 0.14526051134446816" rpy="0.03532604804076814 -0.06496716953483635 -0.05511706101973044"/>
+    <origin xyz="0.048 0.0 0.171" rpy="0.0 0.0 0.0"/>
     <parent link="head_plate_frame"/>
     <child link="azure_kinect_camera_base"/>
@@ -1584,10 +1584,58 @@
     <color rgba="0.9 0.9 0.9 1.0"/>
   </material>
-  <link name="pixel_6_pro"/>
-  <link name="pixel_6_pro/camera_bar"/>
-  <link name="pixel_6_pro/main_camera"/>
-  <link name="pixel_6_pro/ultra_wide_camera"/>
-  <link name="pixel_6_pro/tele_camera"/>
-  <link name="pixel_6_pro/flash_led"/>
+  <link name="pixel_6_pro">
+    <visual>
+      <origin xyz="0.0 0.0 0.0" rpy="0.0 1.5707963267948966 3.141592653589793"/>
+      <geometry>
+        <mesh filename="package://tams_pr2_description/meshes/pixel_6_pro.stl" scale="0.001 0.001 0.001"/>
+      </geometry>
+      <material name="pixel_6_pro_white"/>
+    </visual>
+  </link>
+  <link name="pixel_6_pro/camera_bar">
+    <visual>
+      <origin xyz="0.0 0.0 0.0" rpy="0 0 0"/>
+      <geometry>
+        <box size="0.003 0.022 0.071"/>
+      </geometry>
+      <material name="pixel_6_pro_black"/>
+    </visual>
+  </link>
+  <link name="pixel_6_pro/main_camera">
+    <visual>
+      <origin xyz="0.0 0.0 0.0" rpy="0 0 0"/>
+      <geometry>
+        <cylinder radius="0.0016" length="0.0005"/>
+      </geometry>
+      <material name="pixel_6_pro_grey"/>
+    </visual>
+  </link>
+  <link name="pixel_6_pro/ultra_wide_camera">
+    <visual>
+      <origin xyz="0.0 0.0 0.0" rpy="0 0 0"/>
+      <geometry>
+        <cylinder radius="0.0012" length="0.0005"/>
+      </geometry>
+      <material name="pixel_6_pro_grey"/>
+    </visual>
+  </link>
+  <link name="pixel_6_pro/tele_camera">
+    <visual>
+      <origin xyz="0.0 0.0 0.0" rpy="0 0 0"/>
+      <geometry>
+        <box size="0.004 0.0055 0.0005"/>
+      </geometry>
+      <material name="pixel_6_pro_grey"/>
+    </visual>
+  </link>
+  <link name="pixel_6_pro/flash_led">
+    <visual>
+      <origin xyz="0.0 0.0 0.0" rpy="0 0 0"/>
+      <geometry>
+        <cylinder radius="0.00165" length="0.0005"/>
+      </geometry>
+      <material name="pixel_6_pro_white"/>
+    </visual>
+  </link>
   <joint name="pixel_6_pro/camera_bar_joint" type="fixed">
     <origin xyz="0.00595 -0.0534 0.0" rpy="0.0 0.0 0.0"/>
@@ -1620,5 +1668,15 @@
     <child link="pixel_6_pro"/>
   </joint>
-  <link name="pixel_6_pro_holder"/>
+  <link name="pixel_6_pro_holder">
+    <visual>
+      <origin xyz="0.0 0.0 0.0" rpy="0.0 0.0 1.571"/>
+      <geometry>
+        <mesh filename="package://tams_pr2_description/meshes/pr2_pixel_6_pro_holder_v3.stl" scale="0.001 0.001 0.001"/>
+      </geometry>
+      <material name="pixel_6_pro_holder_material_white">
+        <color rgba="0.95 0.95 0.95 1.0"/>
+      </material>
+    </visual>
+  </link>
   <joint name="pixel_6_pro_holder_joint" type="fixed">
     <origin xyz="-0.0635 0.0 0.0505" rpy="0.0 0.0 0.0"/>
@@ -1755,5 +1813,5 @@
   </transmission>
   <joint name="r_shoulder_pan_joint" type="revolute">
-    <origin xyz="0.0 -0.188 0.0" rpy="0.0 0.0 -0.030585949105467303"/>
+    <origin xyz="0.0 -0.188 0.0" rpy="0.0 0.0 0.0"/>
     <axis xyz="0.0 0.0 1.0"/>
     <parent link="torso_lift_link"/>
@@ -1762,5 +1820,5 @@
     <dynamics damping="10.0"/>
     <safety_controller k_velocity="10.0" k_position="100.0" soft_lower_limit="-2.1353981633974484" soft_upper_limit="0.5646018366025517"/>
-    <calibration rising="-0.77025497063339" falling="0"/>
+    <calibration rising="-0.74550427" falling="0"/>
   </joint>
   <link name="r_shoulder_pan_link">
@@ -1785,5 +1843,5 @@
   </link>
   <joint name="r_shoulder_lift_joint" type="revolute">
-    <origin xyz="0.1 0.0 0.0" rpy="0.0 -0.02932552843059411 0.0"/>
+    <origin xyz="0.1 0.0 0.0" rpy="0.0 0.0 0.0"/>
     <axis xyz="0.0 1.0 0.0"/>
     <parent link="r_shoulder_pan_link"/>
@@ -1792,5 +1850,5 @@
     <dynamics damping="10.0"/>
     <safety_controller k_velocity="10.0" k_position="100.0" soft_lower_limit="-0.3535999999999999" soft_upper_limit="1.2963"/>
-    <calibration rising="0" falling="0.017560181253305468"/>
+    <calibration rising="0" falling="0.02804656"/>
   </joint>
   <link name="r_shoulder_lift_link">
@@ -1815,5 +1873,5 @@
   </link>
   <joint name="r_upper_arm_roll_joint" type="revolute">
-    <origin xyz="0.0 0.0 0.0" rpy="-0.018258450538204244 0.0 0.0"/>
+    <origin xyz="0.0 0.0 0.0" rpy="0.0 0.0 0.0"/>
     <axis xyz="1.0 0.0 0.0"/>
     <parent link="r_shoulder_lift_link"/>
@@ -1822,5 +1880,5 @@
     <dynamics damping="0.1"/>
     <safety_controller k_velocity="2.0" k_position="100.0" soft_lower_limit="-3.7500000000000004" soft_upper_limit="0.65"/>
-    <calibration rising="-1.5713770108738667" falling="0"/>
+    <calibration rising="-1.5587278" falling="0"/>
   </joint>
   <link name="r_upper_arm_roll_link">
@@ -1923,5 +1981,5 @@
   </gazebo>
   <joint name="r_forearm_roll_joint" type="continuous">
-    <origin xyz="0.0 0.0 0.0" rpy="-0.1843833813901606 0.0 0.0"/>
+    <origin xyz="0.0 0.0 0.0" rpy="0.0 0.0 0.0"/>
     <axis xyz="1.0 0.0 0.0"/>
     <parent link="r_elbow_flex_link"/>
@@ -1930,5 +1988,5 @@
     <dynamics damping="0.1"/>
     <safety_controller k_velocity="1.0" k_position="0" soft_lower_limit="0" soft_upper_limit="0"/>
-    <calibration rising="-0.06624517283358188" falling="0"/>
+    <calibration rising="0.0015972" falling="0"/>
   </joint>
   <link name="r_forearm_roll_link">
@@ -1969,5 +2027,5 @@
   </transmission>
   <joint name="r_elbow_flex_joint" type="revolute">
-    <origin xyz="0.4 0.0 0.0" rpy="0.0 0.002147718078060532 0.0"/>
+    <origin xyz="0.4 0.0 0.0" rpy="0.0 0.0 0.0"/>
     <axis xyz="0.0 1.0 0.0"/>
     <parent link="r_upper_arm_link"/>
@@ -1976,5 +2034,5 @@
     <dynamics damping="1.0"/>
     <safety_controller k_velocity="3.0" k_position="100.0" soft_lower_limit="-2.1212999999999997" soft_upper_limit="-0.15"/>
-    <calibration rising="0" falling="-1.1863535155814202"/>
+    <calibration rising="0" falling="-1.15635323"/>
   </joint>
   <link name="r_elbow_flex_link">
@@ -2258,5 +2316,5 @@
   </link>
   <joint name="rh_FFJ4" type="revolute">
-    <origin xyz="0.033 0.0 0.095" rpy="0.0 0.14126182335454857 0.0"/>
+    <origin xyz="0.033 0.0 0.095" rpy="0.0 0.0 0.0"/>
     <axis xyz="0.0 -1.0 0.0"/>
     <parent link="rh_palm"/>
@@ -3519,5 +3577,5 @@
   </gazebo>
   <joint name="l_shoulder_pan_joint" type="revolute">
-    <origin xyz="0.0 0.188 0.0" rpy="0.0 0.0 -0.034817290760945765"/>
+    <origin xyz="0.0 0.188 0.0" rpy="0.0 0.0 0.0"/>
     <axis xyz="0.0 0.0 1.0"/>
     <parent link="torso_lift_link"/>
@@ -3526,5 +3584,5 @@
     <dynamics damping="10.0"/>
     <safety_controller k_velocity="10.0" k_position="100.0" soft_lower_limit="-0.5646018366025517" soft_upper_limit="2.1353981633974484"/>
-    <calibration rising="0.7934907719137071" falling="0"/>
+    <calibration rising="0.82833099" falling="0"/>
   </joint>
   <link name="l_shoulder_pan_link">
@@ -3549,5 +3607,5 @@
   </link>
   <joint name="l_shoulder_lift_joint" type="revolute">
-    <origin xyz="0.1 0.0 0.0" rpy="0.0 -0.04593202341840259 0.0"/>
+    <origin xyz="0.1 0.0 0.0" rpy="0.0 0.0 0.0"/>
     <axis xyz="0.0 1.0 0.0"/>
     <parent link="l_shoulder_pan_link"/>
@@ -3556,5 +3614,5 @@
     <dynamics damping="10.0"/>
     <safety_controller k_velocity="10.0" k_position="100.0" soft_lower_limit="-0.3535999999999999" soft_upper_limit="1.2963"/>
-    <calibration rising="0" falling="-0.01176747185215518"/>
+    <calibration rising="0" falling="-0.00788445"/>
   </joint>
   <link name="l_shoulder_lift_link">
@@ -3579,5 +3637,5 @@
   </link>
   <joint name="l_upper_arm_roll_joint" type="revolute">
-    <origin xyz="0.0 0.0 0.0" rpy="0.003819578775115014 0.0 0.0"/>
+    <origin xyz="0.0 0.0 0.0" rpy="0.0 0.0 0.0"/>
     <axis xyz="1.0 0.0 0.0"/>
     <parent link="l_shoulder_lift_link"/>
@@ -3586,5 +3644,5 @@
     <dynamics damping="0.1"/>
     <safety_controller k_velocity="2.0" k_position="100.0" soft_lower_limit="-0.65" soft_upper_limit="3.7500000000000004"/>
-    <calibration rising="1.599455120499763" falling="0"/>
+    <calibration rising="1.5890453" falling="0"/>
   </joint>
   <link name="l_upper_arm_roll_link">
@@ -3687,5 +3745,5 @@
   </gazebo>
   <joint name="l_forearm_roll_joint" type="continuous">
-    <origin xyz="0.0 0.0 0.0" rpy="-0.027130027402837164 0.0 0.0"/>
+    <origin xyz="0.0 0.0 0.0" rpy="0.0 0.0 0.0"/>
     <axis xyz="1.0 0.0 0.0"/>
     <parent link="l_elbow_flex_link"/>
@@ -3694,5 +3752,5 @@
     <dynamics damping="0.1"/>
     <safety_controller k_velocity="1.0" k_position="0" soft_lower_limit="0" soft_upper_limit="0"/>
-    <calibration rising="0.013565124033188975" falling="0"/>
+    <calibration rising="0.012567" falling="0"/>
   </joint>
   <link name="l_forearm_roll_link">
@@ -3733,5 +3791,5 @@
   </transmission>
   <joint name="l_elbow_flex_joint" type="revolute">
-    <origin xyz="0.4 0.0 0.0" rpy="0.0 -0.015841758965102523 0.0"/>
+    <origin xyz="0.4 0.0 0.0" rpy="0.0 0.0 0.0"/>
     <axis xyz="0.0 1.0 0.0"/>
     <parent link="l_upper_arm_link"/>
@@ -3740,5 +3798,5 @@
     <dynamics damping="1.0"/>
     <safety_controller k_velocity="3.0" k_position="100.0" soft_lower_limit="-2.1212999999999997" soft_upper_limit="-0.15"/>
-    <calibration rising="0" falling="-1.3373751451068947"/>
+    <calibration rising="0" falling="-1.3022338"/>
   </joint>
   <link name="l_elbow_flex_link">
@@ -3804,5 +3862,5 @@
   </link>
   <joint name="l_wrist_flex_joint" type="revolute">
-    <origin xyz="0.321 0.0 0.0" rpy="0.0 0.024323899430578125 0.0"/>
+    <origin xyz="0.321 0.0 0.0" rpy="0.0 0.0 0.0"/>
     <axis xyz="0.0 1.0 0.0"/>
     <parent link="l_forearm_link"/>
@@ -3811,5 +3869,5 @@
     <dynamics damping="0.1"/>
     <safety_controller k_velocity="4.0" k_position="20.0" soft_lower_limit="-2.0" soft_upper_limit="-0.1"/>
-    <calibration rising="0" falling="-0.5082108976740723"/>
+    <calibration rising="0" falling="-0.5241985"/>
   </joint>
   <link name="l_wrist_flex_link">
@@ -3834,5 +3892,5 @@
   </link>
   <joint name="l_wrist_roll_joint" type="continuous">
-    <origin xyz="0.0 0.0 0.0" rpy="-0.10591448792615889 0.0 0.0"/>
+    <origin xyz="0.0 0.0 0.0" rpy="0.0 0.0 0.0"/>
     <axis xyz="1.0 0.0 0.0"/>
     <parent link="l_wrist_flex_link"/>
@@ -3841,5 +3899,5 @@
     <dynamics damping="0.1"/>
     <safety_controller k_velocity="2.0" k_position="0" soft_lower_limit="0" soft_upper_limit="0"/>
-    <calibration rising="-1.5244533256025736" falling="0"/>
+    <calibration rising="-1.43863392" falling="0"/>
   </joint>
   <link name="l_wrist_roll_link">
@@ -4371,32 +4429,4 @@
     </actuator>
   </transmission>
-  <joint name="touch_probe_cylinder_base_joint" type="fixed">
-    <origin xyz="0.019 0.0 0.0" rpy="0.0 0.0 0.0"/>
-    <parent link="l_gripper_tool_frame"/>
-    <child link="touch_probe_cylinder_base_frame"/>
-  </joint>
-  <link name="touch_probe_cylinder_base_frame"/>
-  <joint name="touch_probe_cylinder_top_joint" type="fixed">
-    <origin xyz="0.02099 0.0 0.0" rpy="0.0 0.0 0.0"/>
-    <parent link="touch_probe_cylinder_base_frame"/>
-    <child link="touch_probe_cylinder_top_frame"/>
-  </joint>
-  <link name="touch_probe_cylinder_top_frame">
-    <visual>
-      <origin xyz="-0.010495 0.0 0.0" rpy="0.0 -1.5707963267948966 0.0"/>
-      <geometry>
-        <cylinder radius="0.002" length="0.02099"/>
-      </geometry>
-      <material name="Grey">
-        <color rgba="0.5 0.5 0.5 1.0"/>
-      </material>
-    </visual>
-    <collision>
-      <origin xyz="-0.010495 0.0 0.0" rpy="0.0 -1.5707963267948966 0.0"/>
-      <geometry>
-        <cylinder radius="0.002" length="0.02099"/>
-      </geometry>
-    </collision>
-  </link>
   <joint name="l_forearm_cam_frame_joint" type="fixed">
     <origin xyz="0.135 0.0 0.044" rpy="-1.5707963267948966 -0.5628686837681712 0.0"/>

File: tams_pr2_atom_calibration/urdf/optimized_w_pattern.urdf.xacro (robot description, xacro)
@@ -1552,5 +1552,5 @@
   </joint>
   <joint name="azure_kinect_camera_base_joint" type="fixed">
-    <origin xyz="0.04797663865993433 -0.008366640694689446 0.14526051134446816" rpy="0.03532604804076814 -0.06496716953483635 -0.05511706101973044"/>
+    <origin xyz="0.09443919908378173 0.010873822309647299 0.1675598749914739" rpy="-0.011229592652682889 -0.036835859973993135 -0.011355891320667735"/>
     <parent link="head_plate_frame"/>
     <child link="azure_kinect_camera_base"/>
@@ -4455,3 +4455,31 @@
     <material>PR2/Blue</material>
   </gazebo>
+  <link name="pattern_link">
+    <origin xyz="0 0 0" rpy="0 0 0"/>
+    <visual name="pattern_1_visual">
+      <origin xyz="0 0 0" rpy="0 0 0"/>
+      <geometry>
+        <mesh filename="package://atom_worlds/pattern/models/chessboard_200x214_5x4/chessboard_200x214_5x4.dae"/>
+      </geometry>
+    </visual>
+  </link>
+  <joint name="l_gripper_l_finger_tip_frame-pattern_link" type="fixed">
+    <origin xyz="0.15544173487880106 0.024120168432036276 -0.06851292267149905" rpy="2.9029848739559867 -1.4294167587676068 -1.3284251864282028"/>
+    <parent link="l_gripper_l_finger_tip_frame"/>
+    <child link="pattern_link"/>
+  </joint>
+  <link name="pattern2_link">
+    <origin xyz="0 0 0" rpy="0 0 0"/>
+    <visual name="pattern_2_visual">
+      <origin xyz="0 0 0" rpy="0 0 0"/>
+      <geometry>
+        <mesh filename="package://atom_worlds/pattern/models/chessboard_200x214_5x4/chessboard_200x214_5x4.dae"/>
+      </geometry>
+    </visual>
+  </link>
+  <joint name="rh_forearm-pattern2_link" type="fixed">
+    <origin xyz="-0.036063374240731035 -0.0912910657130159 0.14121449293162777" rpy="-1.5658871902254503 -0.015205289031741136 0.15809811827942563"/>
+    <parent link="rh_forearm"/>
+    <child link="pattern2_link"/>
+  </joint>
 </robot>
